Commit message: Update hw

File: hw1/src/urdf_model/urdf/hw1.urdf (robot description, URDF)
Before this commit: robot hw1, 6 links, 5 joints
Joints:
- removed joint rev1
- removed joint rev2
- removed joint rev3
- removed joint translatory1
- removed joint translatory2
- added joint rev_x: type revolute, parent base_link2, child base_link3, origin xyz=0.0 0.0 0.2 rpy=0.0 0.0 0.0, axis 1 0 0, limit lower=-3.14 upper=3.14 effort=30 velocity=1.0
- added joint rev_y: type revolute, parent base_link3, child base_link4, origin xyz=0.25 0.0 0.0 rpy=0.0 0.0 0.0, axis 0 1 0, limit lower=-3.14 upper=3.14 effort=30 velocity=1.0
- added joint rev_z: type revolute, parent base_link1, child base_link2, origin xyz=0.35 0.00 0.05 rpy=0.0 0.0 0.0, axis 0 0 1, limit lower=-3.14 upper=3.14 effort=30 velocity=1.0
- added joint trans_x: type prismatic, parent base_link, child base_link1, origin xyz=0.0 0.0 0.5 rpy=0.0 0.0 0.0, axis 1 0 0, limit lower=-0.20 upper=0.20 effort=30 velocity=1.0
- added joint trans_z: type prismatic, parent ground_frame, child base_link, origin xyz=0.0 0.0 0.1 rpy=0.0 0.0 0.0, axis 0 0 1, limit lower=-0.3 upper=0.3 effort=30 velocity=1.0

Commit message: Fix revs to wrist

File: hw1/src/urdf_model/urdf/hw1.urdf (robot description, URDF)
Before this commit: robot hw1, 6 links, 5 joints
Links:
- link base_link3: geometry visual cylinder length=0.2 radius=0.1
Joints:
- joint rev_y: origin xyz=0.25 0.0 0.0 rpy=0.0 0.0 0.0 -> xyz=0.2 0.0 0.0 rpy=0.0 0.0 0.0
